File: PCB-1/io.kicad_sch (KiCad schematic)
At the start: 23 parts, among them J1 JST SH 4P., J3 microSD-Card-CTF-11081-P, J4 ZED UART 2, J5 FFC, U13 ISO1541, U2 SR05.TCT, U3 SR05.TCT, U6 SRV05-4, U8 MAX22246CAWA+

Commit message: added photos to docu
Other:
- moved on the sheet: C18, C19, C22, C24, J4, J5, JP1, JP2, R11, TP7, U2, U8
