File: PCB-1/sensors.kicad_sch (KiCad schematic)
At the start: 42 parts, among them J2 JST SH 2, J7 JST SH 2, U1 141352145000, U11 SN74AUP1G17DBVR, U14 MCP23017_ML, U17 141352145000, U18 SN74AUP1G17DBVR, U4 ISM330DHCXTR, U5 BMM150

Commit message: added photos to docu
Other:
- moved on the sheet: C37, C40, C41, C42, R12, R13
