File: PCB-2/io.kicad_sch (KiCad schematic)
At the start: 59 parts, among them J2 USB_C_Receptacle_USB2.0_C3939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, Q1 UMH4NFHATN, U1 SR05.TCT, U19 150060RV75240, U2 USB2514B_Bi, U20 FT231XQ, U3 150060RV75240, U9 FT231XQ, Y1 24MHz

Commit message: added photos to docu
Other:
- moved on the sheet: C40, C41, C42, C43, J2, Q1A, Q1B, R20, R21, R22, R23, R37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
