File: PCB-2/zed.kicad_sch (KiCad schematic)
At the start: 56 parts, among them J3 SMA (GNSS), J5 U.FL, Q3 MBT3906DW1, Q4 AO3400A, U11 PI3USB4002AQ, U13 SN74LVC3G07YZPR, U17 74CBTLV3306GTX, U18 74CBTLV3306GTX, U5 74CBTLV3244BQ,115, U6 ZED-F9P

Commit message: added photos to docu
Connections:
- net REF: now reaches C28.2, U11.6 (REF)
Changed lines of the file:
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@@
     (effects (font (size 0.6 0.6)) (justify left bottom))
+  )
+  (label "REF" (at 71.12 66.04 180)
+    (effects (font (size 0.6 0.6)) (justify right bottom))
   )
   (label "~{EN_ZED_IO}" (at 124.46 204.47 180)
